Commit message: changed gripper limits

File: TRLC-DK1-Follower.urdf (robot description, URDF)
Before this commit: robot TRLC-DK1-Follower, 9 links, 8 joints
Joints:
- removed joint Base_Joint
- removed joint Gripper_Rot
- removed joint Joint_2
- removed joint Joint_3
- removed joint Joint_4
- removed joint Joint_5
- added joint joint1: type revolute, parent base_link, child link1-2, origin xyz=0 0 0.06 rpy=0 0 0, axis 0 0 1, limit lower=-2.0943951023931953 upper=2.0943951023931953 effort=100 velocity=3
- added joint joint2: type revolute, parent link1-2, child Link1, origin xyz=0 0.02 0.0385 rpy=0 0 0, axis 1 0 0, limit lower=-3.141592653589793 upper=0 effort=100 velocity=3
- added joint joint3: type revolute, parent Link1, child Link_2, origin xyz=0 -0.264 0 rpy=0 0 0, axis 1 0 0, limit lower=0 upper=4.71238898038469 effort=100 velocity=3
- added joint joint4: type revolute, parent Link_2, child link4-5, origin xyz=0 0.244004 0.059971 rpy=0 0 0, axis 1 0 0, limit lower=-1.5707963267948966 upper=1.5707963267948966 effort=20 velocity=3
- added joint joint5: type revolute, parent link4-5, child link5-6, origin xyz=0 0.061993 0.038 rpy=0 0 0, axis 0 0 -1, limit lower=-1.57 upper=1.5707963267948966 effort=20 velocity=3
- added joint joint6: type revolute, parent link5-6, child Link6-7, origin xyz=0.0 0.032 -0.0375 rpy=0 0 0, axis 0 1 0, limit lower=-3.141592653589793 upper=3.141592653589793 effort=20 velocity=3
- joint gripper_left: limit lower=0.0 upper=0.04 effort=0 velocity=0 -> lower=-0.045 upper=0.0 effort=20 velocity=0.2; origin xyz=0 0 0 rpy=0 0 0 -> xyz=-0.04 0 0 rpy=0 0 0
- joint gripper_right: limit lower=0.0 upper=0.04 effort=0 velocity=0 -> lower=-0.045 upper=0.0 effort=20 velocity=0.2; origin xyz=0 0 0 rpy=0 0 0 -> xyz=0.04 0 0 rpy=0 0 0

Commit message: update meshes and joint xyz offsets

File: TRLC-DK1-Follower.urdf (robot description, URDF)
Before this commit: robot TRLC-DK1-Follower, 9 links, 8 joints
Joints:
- joint joint1: origin xyz=0 0 0.06 rpy=0 0 0 -> xyz=0 0 0.0615 rpy=0 0 0
- joint joint5: origin xyz=0 0.061993 0.038 rpy=0 0 0 -> xyz=0 0.061993 0.0375 rpy=0 0 0
- joint joint6: origin xyz=0.0 0.032 -0.0375 rpy=0 0 0 -> xyz=0.0 0.032 -0.0425 rpy=0 0 0

Commit message: add dae versions of first 3 links

File: TRLC-DK1-Follower.urdf (robot description, URDF)
Before this commit: robot TRLC-DK1-Follower, 9 links, 8 joints
Links:
- link Link1: geometry collision mesh filename=meshes/Link1.stl; visual mesh filename=meshes/link1.dae
- link base_link: geometry collision mesh filename=meshes/base_link.stl; visual mesh filename=meshes/base_link.dae
- link link1-2: geometry collision mesh filename=meshes/link1-2.stl; visual mesh filename=meshes/link1-2.dae

Commit message: add link 2 & link4-5 dae versions

File: TRLC-DK1-Follower.urdf (robot description, URDF)
Before this commit: robot TRLC-DK1-Follower, 9 links, 8 joints
Links:
- link Link_2: geometry collision mesh filename=meshes/Link_2.stl; visual mesh filename=meshes/link2.dae
- link link4-5: geometry collision mesh filename=meshes/link4-5.stl; visual mesh filename=meshes/link4-5.dae

Commit message: complete visuals for wrist

File: TRLC-DK1-Follower.urdf (robot description, URDF)
Before this commit: robot TRLC-DK1-Follower, 9 links, 8 joints
Links:
- link Link6-7: geometry collision mesh filename=meshes/Link6-7.stl; visual mesh filename=meshes/link6-7.dae
- link finger_left: geometry collision mesh filename=meshes/finger_left.stl; visual mesh filename=meshes/finger_left.dae
- link finger_right: geometry collision mesh filename=meshes/finger_right.stl; visual mesh filename=meshes/finger_right.dae
- link link5-6: geometry collision mesh filename=meshes/link5-6.stl; visual mesh filename=meshes/link5-6.dae
Joints:
- joint gripper_left: origin xyz=-0.04 0 0 rpy=0 0 0 -> xyz=0 0 0 rpy=0 0 0
- joint gripper_right: origin xyz=0.04 0 0 rpy=0 0 0 -> xyz=0 0 0 rpy=0 0 0
- joint joint5: origin xyz=0 0.061993 0.0375 rpy=0 0 0 -> xyz=0 0.061868 0.0425 rpy=0 0 0

Commit message: define tool0 TCP

File: TRLC-DK1-Follower.urdf (robot description, URDF)
Before this commit: robot TRLC-DK1-Follower, 9 links, 8 joints
Links:
- added link tool0
Joints:
- added joint gripper_tool0: type fixed, parent Link6-7, child tool0, origin xyz=0 0.158 0 rpy=-1.5707963267948966 0 0

Commit message: fix range precision

File: TRLC-DK1-Follower.urdf (robot description, URDF)
Before this commit: robot TRLC-DK1-Follower, 10 links, 9 joints
Joints:
- joint joint5: limit lower=-1.57 upper=1.5707963267948966 effort=20 velocity=3 -> lower=-1.5707963267948966 upper=1.5707963267948966 effort=20 velocity=3

Commit message: add mass values provided by Aakaar

File: TRLC-DK1-Follower.urdf (robot description, URDF)
Before this commit: robot TRLC-DK1-Follower, 10 links, 9 joints
Links:
- link Link1: mass 0.537601776973517 -> 0.55
- link Link6-7: mass 0.289722572316062 -> 0.45775
- link Link_2: mass 0.299922094541001 -> 0.54467
- link base_link: mass 0.02782 -> 0.21
- link finger_left: mass 0.0745959905268717 -> 0.037299
- link finger_right: mass 0.0745959905268717 -> 0.037299
- link link1-2: mass 0.024532 -> 0.09
- link link4-5: mass 0.0142938416889126 -> 0.361
- link link5-6: mass 0.11909711022403 -> 0.35879

Commit message: use separate collision & visual folders for meshes

File: TRLC-DK1-Follower.urdf (robot description, URDF)
Before this commit: robot TRLC-DK1-Follower, 10 links, 9 joints
Links:
- removed link Link1
- removed link Link6-7
- removed link Link_2
- added link link1, mass 0.55; collision mesh filename=meshes/collision/link1.stl; visual mesh filename=meshes/visual/link1.dae
- added link link2, mass 0.54467; collision mesh filename=meshes/collision/link2.stl; visual mesh filename=meshes/visual/link2.dae
- added link link6-7, mass 0.45775; collision mesh filename=meshes/collision/link6-7.stl; visual mesh filename=meshes/visual/link6-7.dae
- link base_link: geometry collision mesh filename=meshes/collision/base_link.stl; visual mesh filename=meshes/visual/base_link.dae
- link finger_left: geometry collision mesh filename=meshes/collision/finger_left.stl; visual mesh filename=meshes/visual/finger_left.dae
- link finger_right: geometry collision mesh filename=meshes/collision/finger_right.stl; visual mesh filename=meshes/visual/finger_right.dae
- link link1-2: geometry collision mesh filename=meshes/collision/link1-2.stl; visual mesh filename=meshes/visual/link1-2.dae
- link link4-5: geometry collision mesh filename=meshes/collision/link4-5.stl; visual mesh filename=meshes/visual/link4-5.dae
- link link5-6: geometry collision mesh filename=meshes/collision/link5-6.stl; visual mesh filename=meshes/visual/link5-6.dae
Joints:
- joint gripper_left: parent Link6-7 -> link6-7
- joint gripper_right: parent Link6-7 -> link6-7
- joint gripper_tool0: parent Link6-7 -> link6-7
- joint joint2: child Link1 -> link1
- joint joint3: child Link_2 -> link2; parent Link1 -> link1
- joint joint4: parent Link_2 -> link2
- joint joint6: child Link6-7 -> link6-7

Commit message: change to x forward, use glb, add inertia

File: TRLC-DK1-Follower.urdf (robot description, URDF)
Before this commit: robot TRLC-DK1-Follower, 10 links, 9 joints
Links:
- removed link link1
- removed link link2
- added link link2-3, mass 1.0; collision mesh filename=meshes/collision/link2-3.stl; visual mesh filename=meshes/visual/link2-3.glb
- added link link3-4, mass 0.54467; collision mesh filename=meshes/collision/link3-4.stl; visual mesh filename=meshes/visual/link3-4.glb
- link base_link: geometry collision mesh filename=meshes/collision/base_link.stl; visual mesh filename=meshes/visual/base_link.glb
- link finger_left: geometry collision mesh filename=meshes/collision/finger_left.stl; visual mesh filename=meshes/visual/finger_left.glb
- link finger_right: geometry collision mesh filename=meshes/collision/finger_right.stl; visual mesh filename=meshes/visual/finger_right.glb
- link link1-2: geometry collision mesh filename=meshes/collision/link1-2.stl; visual mesh filename=meshes/visual/link1-2.glb
- link link4-5: geometry collision mesh filename=meshes/collision/link4-5.stl; visual mesh filename=meshes/visual/link4-5.glb
- link link5-6: geometry collision mesh filename=meshes/collision/link5-6.stl; visual mesh filename=meshes/visual/link5-6.glb
- link link6-7: geometry collision mesh filename=meshes/collision/link6-7.stl; visual mesh filename=meshes/visual/link6-7.glb
Joints:
- joint gripper_left: axis -1 0 0 -> 0 1 0; limit lower=-0.045 upper=0.0 effort=20 velocity=0.2 -> lower=-0.045 upper=0.001 effort=20 velocity=0.2
- joint gripper_right: axis 1 0 0 -> 0 -1 0; limit lower=-0.045 upper=0.0 effort=20 velocity=0.2 -> lower=-0.045 upper=0.001 effort=20 velocity=0.2; mimic joint=gripper_left multiplier=1 offset=0 -> (none)
- joint gripper_tool0: origin xyz=0 0.158 0 rpy=-1.5707963267948966 0 0 -> xyz=0.158 0 0 rpy=-1.5707963267948966 0 -1.5707963267948966
- joint joint2: axis 1 0 0 -> 0 -1 0; child link1 -> link2-3; limit lower=-3.141592653589793 upper=0 effort=100 velocity=3 -> lower=-3.141592653589793 upper=0.001 effort=100 velocity=3; origin xyz=0 0.02 0.0385 rpy=0 0 0 -> xyz=0.02 0.0/ 0.0385 rpy=0 0 0
- joint joint3: axis 1 0 0 -> 0 -1 0; child link2 -> link3-4; limit lower=0 upper=4.71238898038469 effort=100 velocity=3 -> lower=-0.001 upper=4.71238898038469 effort=100 velocity=3; origin xyz=0 -0.264 0 rpy=0 0 0 -> xyz=-0.264 0 0 rpy=0 0 0; parent link1 -> link2-3
- joint joint4: axis 1 0 0 -> 0 -1 0; origin xyz=0 0.244004 0.059971 rpy=0 0 0 -> xyz=0.244004 0 0.059971 rpy=0 0 0; parent link2 -> link3-4
- joint joint5: origin xyz=0 0.061868 0.0425 rpy=0 0 0 -> xyz=0.061868 0 0.0425 rpy=0 0 0
- joint joint6: axis 0 1 0 -> 1 0 0; origin xyz=0.0 0.032 -0.0425 rpy=0 0 0 -> xyz=0.032 0 -0.0425 rpy=0 0 0

Commit message: add cam link

File: TRLC-DK1-Follower.urdf (robot description, URDF)
Before this commit: robot TRLC-DK1-Follower, 10 links, 9 joints
Links:
- added link camera; visual cylinder length=0.015 radius=0.008
- added link camera_base; visual box size=0.03 0.025 0.015
Joints:
- added joint camera_joint: type fixed, parent camera_base, child camera, origin xyz=0.01 0.0 0.0 rpy=0 0 0
- added joint hand_to_camera_mount: type fixed, parent link6-7, child camera_base, origin xyz=0.035 0 0.0675 rpy=0 0.3491 0

Commit message: fix joint2 xyz

File: TRLC-DK1-Follower.urdf (robot description, URDF)
Before this commit: robot TRLC-DK1-Follower, 12 links, 11 joints
Joints:
- joint camera_joint: origin xyz=0.01 0.0 0.0 rpy=0 0 0 -> xyz=0.01 0 0 rpy=0 0 0
- joint joint2: origin xyz=0.02 0.0/ 0.0385 rpy=0 0 0 -> xyz=0.02 0 0.0385 rpy=0 0 0

Commit message: remove material, simplify cam

File: TRLC-DK1-Follower.urdf (robot description, URDF)
Before this commit: robot TRLC-DK1-Follower, 12 links, 11 joints
Links:
- removed link camera_base
- link camera: geometry 
Joints:
- removed joint hand_to_camera_mount
- joint camera_joint: origin xyz=0.01 0 0 rpy=0 0 0 -> xyz=0.0471 0 0.063314 rpy=0 0.2618 0; parent camera_base -> link6-7
- joint joint2: origin xyz=0.02 0 0.0385 rpy=0 0 0 -> xyz=0.02 0.0 0.0385 rpy=0 0 0

Commit message: avoid joint limits too close to home pose

File: TRLC-DK1-Follower.urdf (robot description, URDF)
Before this commit: robot TRLC-DK1-Follower, 11 links, 10 joints
Joints:
- joint joint2: limit lower=-3.141592653589793 upper=0.001 effort=100 velocity=3 -> lower=-3.141592653589793 upper=0.01 effort=100 velocity=3
- joint joint3: limit lower=-0.001 upper=4.71238898038469 effort=100 velocity=3 -> lower=-0.01 upper=4.71238898038469 effort=100 velocity=3

Commit message: update max velocity

File: TRLC-DK1-Follower.urdf (robot description, URDF)
Before this commit: robot TRLC-DK1-Follower, 11 links, 10 joints
Joints:
- joint gripper_left: limit lower=-0.045 upper=0.001 effort=20 velocity=0.2 -> lower=-0.045 upper=0.001 effort=20 velocity=0.18
- joint gripper_right: limit lower=-0.045 upper=0.001 effort=20 velocity=0.2 -> lower=-0.045 upper=0.001 effort=20 velocity=0.18
- joint joint1: limit lower=-2.0943951023931953 upper=2.0943951023931953 effort=100 velocity=3 -> lower=-2.0943951023931953 upper=2.0943951023931953 effort=100 velocity=5.4
- joint joint2: limit lower=-3.141592653589793 upper=0.01 effort=100 velocity=3 -> lower=-3.141592653589793 upper=0.01 effort=100 velocity=5.4
- joint joint3: limit lower=-0.01 upper=4.71238898038469 effort=100 velocity=3 -> lower=-0.01 upper=4.71238898038469 effort=100 velocity=5.4
- joint joint4: limit lower=-1.5707963267948966 upper=1.5707963267948966 effort=20 velocity=3 -> lower=-1.5707963267948966 upper=1.5707963267948966 effort=20 velocity=5.4
- joint joint5: limit lower=-1.5707963267948966 upper=1.5707963267948966 effort=20 velocity=3 -> lower=-1.5707963267948966 upper=1.5707963267948966 effort=20 velocity=5.4
- joint joint6: limit lower=-3.141592653589793 upper=3.141592653589793 effort=20 velocity=3 -> lower=-3.141592653589793 upper=3.141592653589793 effort=20 velocity=5.4

Commit message: increase joint range of joint4 to allow higher orthogonal eef pose

File: TRLC-DK1-Follower.urdf (robot description, URDF)
Before this commit: robot TRLC-DK1-Follower, 11 links, 10 joints
Joints:
- joint joint4: limit lower=-1.5707963267948966 upper=1.5707963267948966 effort=20 velocity=5.4 -> lower=-1.95 upper=1.5707963267948966 effort=20 velocity=5.4

Commit message: add corrected mass values provided by Aakaar

File: TRLC-DK1-Follower.urdf (robot description, URDF)
Before this commit: robot TRLC-DK1-Follower, 11 links, 10 joints
Links:
- link base_link: mass 0.21 -> 0.4455
- link finger_left: mass 0.037299 -> 0.05
- link finger_right: mass 0.037299 -> 0.05
- link link1-2: mass 0.09 -> 0.0886
- link link2-3: mass 1.0 -> 1.0327
- link link3-4: mass 0.54467 -> 0.6073
- link link4-5: mass 0.361 -> 0.4232
- link link5-6: mass 0.35879 -> 0.4214
- link link6-7: mass 0.45775 -> 0.8506

Commit message: fix joint2 rotation axis

File: TRLC-DK1-Follower.urdf (robot description, URDF)
Before this commit: robot TRLC-DK1-Follower, 11 links, 10 joints
Joints:
- joint joint2: axis 0 -1 0 -> 0 1 0; limit lower=-3.141592653589793 upper=0.01 effort=100 velocity=5.4 -> lower=-0.01 upper=3.141592653589793 effort=100 velocity=5.4

Commit message: local urdf fixes

File: TRLC-DK1-Follower.urdf (robot description, URDF)
Before this commit: robot TRLC-DK1-Follower, 11 links, 10 joints
Links:
- link link3-4: mass 0.6073 -> 0.5
- link link5-6: mass 0.4214 -> 0.35
- link link6-7: mass 0.8506 -> 0.65

Commit message: new mass values

File: TRLC-DK1-Follower.urdf (robot description, URDF)
Before this commit: robot TRLC-DK1-Follower, 11 links, 10 joints
Links:
- link base_link: mass 0.4455 -> 0.5111
- link link1-2: mass 0.0886 -> 0.5965
- link link2-3: mass 1.0327 -> 0.9084
- link link3-4: mass 0.5 -> 0.7089
- link link4-5: mass 0.4232 -> 0.3995
- link link5-6: mass 0.35 -> 0.4121
- link link6-7: mass 0.65 -> 0.5
